File: PCBA/Forker.kicad_sch (KiCad schematic)
At the start: 47 parts, among them J1 USB C, J11 Conn_01x05, J12 Conn_02x06_Odd_Even, J2 Conn_01x02, J3 Conn_01x06, J4 AA, J5 AA, J6 Conn_01x02, J7 Conn_01x02, J8 Conn_01x02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

Commit message: Update PCB Layout
Parts:
- removed J2, J9: Conn_01x02, Connector_PinHeader_2.54mm:PinHeader_1x02_P2.54mm_Vertical, symbol Connector_Generic:Conn_01x02
- removed U8: HL118, Local_Footprints:SOP-8-1EP_3.9x4.9mm_P1.27mm_EP2.4x3.3mm, symbol -Local_Lib:Integrated Circuits/IC-000005
- added JP2, JP3, JP4: SolderJumper_2_Open, Jumper:SolderJumper-2_P1.3mm_Open_TrianglePad1.0x1.5mm, symbol Jumper:SolderJumper_2_Open
Connections:
- net GND: now also R4.1, JP2.2 (B), JP3.2 (B), JP4.2 (B)
- net at R11.1, U3.14 (PA18/A7/BSL): no longer U6.3 (INB)
- net at U3.13 (PA17): now also U6.3 (INB); no longer U7.2 (INA)
- net at U3.10 (PA6): now also U7.2 (INA); no longer U7.3 (INB)
- net at U3.9 (PA4): now also U7.3 (INB)
- net at U1.1 (TS): now also R4.2
- new net: JP4.1 (A), U7.9 (EP)
- new net: JP3.1 (A), U6.9 (EP)
- new net: JP2.1 (A), U5.9 (EP)
Other:
- moved on the sheet: J6, J7, J8, R4

Commit message: -Update PCBA connector location -Add cutouts for PCBA -Add Mounting Holes
Parts:
- removed JP2, JP3, JP4: SolderJumper_2_Open, Jumper:SolderJumper-2_P1.3mm_Open_TrianglePad1.0x1.5mm, symbol Jumper:SolderJumper_2_Open
- removed R12, R5, R9: 10k, Resistor_SMD:R_0603_1608Metric_Pad0.98x0.95mm_HandSolder, symbol -Local_Lib:Resistors/RES-000010
- added H1, H2: MountingHole, MountingHole:MountingHole_2.2mm_M2, symbol Mechanical:MountingHole
- added U8: HL118, Local_Footprints:SOP-8-1EP_3.9x4.9mm_P1.27mm_EP2.4x3.3mm, symbol -Local_Lib:Integrated Circuits/IC-000005
Connections:
- net +3V3: now also U8.2 (INA)
- net +5V: now also U4.1 (CE)
- net GND: now also U5.9 (EP), U6.9 (EP), U7.9 (EP), U8.3 (INB), U8.6 (GND), U8.7 (GND), U8.9 (EP)
- net at U6.2 (INA): now also U3.12 (PA16/A8); no longer U3.19 (PA24/A3)
- net at U6.3 (INB): now also U3.19 (PA24/A3); no longer U3.13 (PA17)
- net at R6.1: now also U3.10 (PA6); no longer U3.12 (PA16/A8)
- net at C8.1, D5.1 (K), SW8.1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: now also U8.4 (VDD); no longer L2.1
- net at U7.2 (INA): now also U3.13 (PA17); no longer U3.10 (PA6)
- net at U7.3 (INB): now also U3.11 (PA11); no longer U3.9 (PA4)
- net at R7.1: now also U3.9 (PA4); no longer U3.11 (PA11)
- new net: L2.1, U8.8 (VOUTA)
Other:
- moved on the sheet: C3, C5, D2, D3, R6, R7
